Commit message: wheel_y_offset modified

File: src/my_robot_description/urdf/my_robot_base_mesh.xacro (robot description, xacro)
@@ -1,5 +1,5 @@
 <?xml version="1.0"?>
 <robot xmlns:xacro="http://www.ros.org/wiki/xacro">
-    <xacro:property name="wheel_y_offset" value="0.05807"/>
+    <xacro:property name="wheel_y_offset" value="0.075"/>
     <xacro:property name="wheel_z_offset" value="0.02"/>
     <xacro:property name="wheel_radius" value="0.0325"/>
