Commit message: - Updated RViz configuration () - Modified launch files for joystick and LiDAR (, ) - Removed unused - Adjusted  and base mesh files for compatibility

File: src/my_robot_description/urdf/lidar.xacro (robot description, xacro)
@@ -45,17 +45,22 @@
                     <resolution>0.01</resolution>
                 </range>
+                <noise>
+                    <type>gaussian</type>
+                    <mean>0.0</mean>
+                    <stddev>0.01</stddev>
+                </noise>
             </ray>
-            <plugin name="laser_sensor" filename="libgazebo_ros_ray_sensor.so">
+            <!-- <plugin name="laser_sensor" filename="libgazebo_ros_ray_sensor.so">
                 <ros>
-                    <!-- Configure namespace and remap to publish to /ray/pointcloud2 -->
-                    <argument>--ros-args --remap ~/out:=scan</argument>
-                </ros>
+                    Configure namespace and remap to publish to /ray/pointcloud2
+                    <argument>~/out:=scan</argument>
+                </ros> -->
                 <!-- Output as a PointCloud2, see above for other types -->
-                <output_type>sensor_msgs/LaserScan</output_type>
+                <!-- <output_type>sensor_msgs/LaserScan</output_type> -->
                 <!-- Clip intensity values so all are above 100, optional -->
                 <!-- <min_intensity>100.0</min_intensity> -->
                 <!-- Frame id for header of output, defaults to sensor's parent link name -->
-                <frame_name>laser</frame_name>
-            </plugin>
+                <!-- <frame_name>laser</frame_name>
+            </plugin> -->
         </sensor>
     </gazebo>

File: src/my_robot_description/urdf/my_robot.urdf.xacro (robot description, xacro)
@@ -7,5 +7,5 @@
     <xacro:include filename="my_robot_base_mesh.xacro" />
     <xacro:include filename="lidar.xacro" />
-    <xacro:include filename="gyroscope.xacro" />
+    <xacro:include filename="imu.xacro" />
     <!-- <xacro:include filename="my_robot_gazebo_control.xacro" /> -->
     <xacro:include filename="my_robot_ros2_control.xacro" />

File: src/my_robot_description/urdf/my_robot_base_mesh.xacro (robot description, xacro)
@@ -15,8 +15,8 @@
     <xacro:property name="lidar_radius" value="0.0278"/>
     <xacro:property name="lidar_length" value="0.0413"/>
-    <xacro:property name="gyroscope_length" value="0.015"/>
-    <xacro:property name="gyroscope_width" value="0.02"/>
-    <xacro:property name="gyroscope_height" value="0.002"/>
-    <xacro:property name="body_gyroscope_z_distance" value="${body_length - 0.046}"/>
+    <xacro:property name="imu_length" value="0.015"/>
+    <xacro:property name="imu_width" value="0.02"/>
+    <xacro:property name="imu_height" value="0.002"/>
+    <xacro:property name="body_imu_z_distance" value="${body_length - 0.046}"/>
     <!-- footprint_link -->
     <link name="footprint_link" />
