Commit message: Clean up my_robot_description package

File: src/my_robot_description/urdf/my_robot.urdf.xacro (robot description, xacro)
@@ -1,6 +1,4 @@
 <?xml version="1.0"?>
 <robot name="my_robot_description" xmlns:xacro="http://www.ros.org/wiki/xacro">
-    <!-- toggle xacro functionality -->
-    <xacro:arg name="use_ros2_control" default="true"/>
     <xacro:include filename="common_properties.xacro" />
     <!-- <xacro:include filename="my_robot_base.xacro" /> -->
@@ -9,11 +7,3 @@
     <xacro:include filename="lidar.xacro" />
     <xacro:include filename="imu.xacro" />
-    <!-- <xacro:include filename="my_robot_ros2_control.xacro" />   -->
-    <!-- <xacro:include filename="my_robot_gazebo_control.xacro" /> -->
-    <!-- <xacro:if value="$(arg use_ros2_control)">
-        <xacro:include filename="my_robot_ros2_control.xacro" />
-    </xacro:if>
-    <xacro:unless value="$(arg use_ros2_control)">
-    <xacro:include filename="my_robot_gazebo_control.xacro" />
-    </xacro:unless>  -->
 </robot>

File: src/my_robot_description/urdf/my_robot_base_mesh.xacro (robot description, xacro)
@@ -19,4 +19,5 @@
     <xacro:property name="imu_height" value="0.0015"/>
     <xacro:property name="base_imu_z_distance" value="${body_length - 0.046}"/>
+    <xacro:property name= "meshes_file_direction" value="package://my_robot_description/models/meshes"/>
     <!-- base_footprint -->
     <link name="base_footprint" />
@@ -25,5 +26,5 @@
         <visual>
             <geometry>
-                <mesh filename="package://my_robot_description/models/meshes/my_robot_base.stl" scale="0.001 0.001 0.001"/>
+                <mesh filename="${meshes_file_direction}/my_robot_base.stl" scale="0.001 0.001 0.001"/>
             </geometry>
             <material name="grünlichesGrau"/>
@@ -36,5 +37,5 @@
             <origin xyz="0.0 0.0 ${body_length / 2}" rpy="0.0 0.0 0.0"/>
         </collision>
-        <xacro:box_inertia m="1000.0" l="${body_length}" w="${body_radius * 2}" h="${body_radius * 2}"
+        <xacro:box_inertia m="2.0" l="${body_length}" w="${body_radius * 2}" h="${body_radius * 2}"
                                 xyz="0.0 0.0 ${wheel_z_offset + (body_length / 2) - 0.02}" rpy="0.0 0.0 0.0" />
     </link>
@@ -50,5 +51,5 @@
             <visual>
                 <geometry>
-                <mesh filename="package://my_robot_description/models/meshes/wheel.stl" scale="0.001 0.001 0.001"/>
+                <mesh filename="${meshes_file_direction}/wheel.stl" scale="0.001 0.001 0.001"/>
                 </geometry>
                 <material name="grauBlau"/>
@@ -61,5 +62,5 @@
                 <origin xyz="0.0 0.0 0.0" rpy="0.0 0.0 0.0"/>
             </collision>
-            <xacro:cylinder_inertia m="500.0" r="${wheel_radius}" h="${wheel_length}"
+            <xacro:cylinder_inertia m="0.5" r="${wheel_radius}" h="${wheel_length}"
                                     xyz="0.0 0.0 0.0" rpy="0.0 0.0 0.0" />
         </link>
@@ -86,5 +87,5 @@
             <visual>
                 <geometry>
-                    <mesh filename="package://my_robot_description/models/meshes/caster_wheel.stl" scale="0.001 0.001 0.001"/>
+                    <mesh filename="${meshes_file_direction}/caster_wheel.stl" scale="0.001 0.001 0.001"/>
                 </geometry>
                 <material name="black"/>
@@ -98,5 +99,5 @@
                 <origin xyz="0.0 0.0 0.0" rpy="0.0 0.0 0.0"/>
             </collision>
-            <xacro:cylinder_inertia m="250.0" r="${caster_wheel_radius}" h="${caster_wheel_length}"
+            <xacro:cylinder_inertia m="0.250" r="${caster_wheel_radius}" h="${caster_wheel_length}"
                                     xyz="0.0 0.0 0.0" rpy="0.0 0.0 0.0" />
         </link>
@@ -130,3 +131,12 @@
         <origin xyz="0 0 0.1" rpy="0 0 0"/>
     </joint> -->
+    <!-- <plugin name="joint_state_publisher" filename="libgazebo_ros_joint_state_publisher.so">
+    <ros>
+        <robotNamespace>/my_robot</robotNamespace>
+        <jointName>base_left_wheel_joint, base_right_wheel_joint</jointName>
+        <remapping>joint_states:=/joint_states</remapping>
+        <updateRate>100.0</updateRate>
+        <alwaysOn>true</alwaysOn>
+    </ros>
+    </plugin> -->
 </robot>
