Commit message: rename body- and footprint-link to base_link and base_footprint and modify the wheel_seperation

File: src/my_robot_description/urdf/common_properties.xacro (robot description, xacro)
@@ -16,5 +16,8 @@
         <color rgba="0.0 0.0 0.0 1"/>
     </material>
-    <gazebo reference="body_link">
+    <material name="green">
+        <color rgba="0.0 0.1 0.0 1"/>
+    </material>
+    <gazebo reference="base_link">
         <material>Gazebo/DarkGrey</material>
     </gazebo>

File: src/my_robot_description/urdf/imu.xacro (robot description, xacro)
@@ -7,5 +7,5 @@
                 <box size="${imu_length} ${imu_width} ${imu_height}"/>
             </geometry>
-            <material name="red"/>
+            <material name="green"/>
             <origin xyz="0.0 0.0 ${imu_height/2}" rpy="0.0 0.0 ${pi/2}"/>
         </visual>
@@ -19,9 +19,9 @@
                                 xyz="0.0 0.0 ${imu_height/2}" rpy="0.0 0.0 0.0" />
     </link>
-    <!-- body_imu_joint -->
-    <joint name="body_imu_joint" type="fixed">
-        <parent link="body_link"/>
+    <!-- base_imu_joint -->
+    <joint name="base_imu_joint" type="fixed">
+        <parent link="base_link"/>
         <child link="bno055"/>
-        <origin xyz="${-body_radius + imu_length} 0 ${body_imu_z_distance}" rpy= "0 0 0"/>
+        <origin xyz="0 0 ${base_imu_z_distance + 0.0345}" rpy= "0 0 0"/>
     </joint>
     <gazebo reference="bno055">
@@ -39,4 +39,5 @@
                     <remapping>~/out:=/imu/data</remapping>
                 </ros>
+                <frame_id>bno055</frame_id>
             </plugin>
             <imu>

File: src/my_robot_description/urdf/lidar.xacro (robot description, xacro)
@@ -19,11 +19,11 @@
                                 xyz="0.0 0.0 ${lidar_length/2}" rpy="0.0 0.0 0.0" />
     </link>
-    <!-- body_laser_joint -->
-    <joint name="body_laser_joint" type="fixed">
-        <parent link="body_link"/>
+    <!-- base_laser_joint -->
+    <joint name="base_laser_joint" type="fixed">
+        <parent link="base_link"/>
         <child link="laser"/>
-        <origin xyz="0 0 ${body_length - 0.002}" rpy= "0 0 0"/>
+        <origin xyz="0 0 ${body_length - 0.0025}" rpy= "0 0 0"/>
     </joint>
-    <gazebo reference="laser">
+    <!-- <gazebo reference="laser">
         <material>Gazebo/Red</material>
         <sensor name="laser" type="ray">
@@ -50,5 +50,5 @@
                     <stddev>0.01</stddev>
                 </noise>
-            </ray>
+            </ray> -->
             <!-- <plugin name="laser_sensor" filename="libgazebo_ros_ray_sensor.so">
                 <ros>
@@ -63,5 +63,5 @@
                 <!-- <frame_name>laser</frame_name>
             </plugin> -->
-        </sensor>
-    </gazebo>
+        <!-- </sensor>
+    </gazebo>     -->
 </robot>

File: src/my_robot_description/urdf/my_robot.urdf.xacro (robot description, xacro)
@@ -9,5 +9,5 @@
     <xacro:include filename="imu.xacro" />
     <!-- <xacro:include filename="my_robot_gazebo_control.xacro" /> -->
-    <xacro:include filename="my_robot_ros2_control.xacro" />
+    <!-- <xacro:include filename="my_robot_ros2_control.xacro" />   -->
     <!-- <xacro:if value="$(arg use_ros2_control)">
         <xacro:include filename="my_robot_ros2_control.xacro" />

File: src/my_robot_description/urdf/my_robot_base.xacro (robot description, xacro)
@@ -5,5 +5,5 @@
     <xacro:property name="wheel_radius" value="0.0325"/>
     <xacro:property name="wheel_length" value="0.025"/>
-    <xacro:property name="robot_center_to_body_link_z_distance" value="0.1375"/>
+    <xacro:property name="robot_center_to_base_link_z_distance" value="0.1375"/>
     <xacro:property name="body_length" value="0.1855"/>
     <xacro:property name="body_radius" value="0.07"/>
@@ -13,11 +13,11 @@
     <xacro:property name="body_caster_wheel_link_distance" value="0.06"/>
     <xacro:property name="body_caster_wheel_Achse_distance" value="0.0025"/>
-    <xacro:property name="body_link_inertia_z_offset" value="0.0925"/>
+    <xacro:property name="base_link_inertia_z_offset" value="0.0925"/>
     <xacro:property name="lidar_radius" value="0.0278"/>
     <xacro:property name="lidar_length" value="0.0413"/>
-    <!-- footprint_link -->
-    <link name="footprint_link" />
-    <!-- body_link -->
-    <link name="body_link">
+    <!-- base_footprint -->
+    <link name="base_footprint" />
+    <!-- base_link -->
+    <link name="base_link">
         <visual>
             <geometry>
@@ -27,5 +27,5 @@
             <material name="grey"/>
             <origin xyz="0.0 0.0 ${wheel_z_offset + (body_length / 2) - 0.02}" rpy="0.0 0.0 0.0"/>
-            <!-- <origin xyz="0.0 0.0 ${robot_center_to_body_link_z_distance}" rpy="${pi/2} 0.0 0.0"/>           -->
+            <!-- <origin xyz="0.0 0.0 ${robot_center_to_base_link_z_distance}" rpy="${pi/2} 0.0 0.0"/>           -->
         </visual>
         <collision>
@@ -35,5 +35,5 @@
             </geometry>
             <origin xyz="0.0 0.0 ${wheel_z_offset + (body_length / 2) - 0.02}" rpy="0.0 0.0 0.0"/>
-            <!-- <origin xyz="0.0 0.0 ${robot_center_to_body_link_z_distance}" rpy="${pi/2} 0.0 0.0"/>                    -->
+            <!-- <origin xyz="0.0 0.0 ${robot_center_to_base_link_z_distance}" rpy="${pi/2} 0.0 0.0"/>                    -->
         </collision>
         <!-- <collision>
@@ -41,15 +41,15 @@
                 <mesh filename="package://my_robot/meshes_description/my_robot.stl" scale="0.001 0.001 0.001"/>
             </geometry>
-            <origin xyz="0.0 0.0 ${robot_center_to_body_link_z_distance}" rpy="${pi/2} 0.0 0.0"/>
+            <origin xyz="0.0 0.0 ${robot_center_to_base_link_z_distance}" rpy="${pi/2} 0.0 0.0"/>
         </collision> -->
         <xacro:box_inertia m="10.0" l="${body_length}" w="${body_radius * 2}" h="${wheel_x_offset * 2}"
                                 xyz="0.0 0.0 ${wheel_z_offset + (body_length / 2) - 0.02}" rpy="0.0 0.0 0.0" />
         <!-- <xacro:cylinder_inertia m="1.5" r="${body_radius}" h="${body_length}"
-                        xyz="0.0 0.0 ${body_link_inertia_z_offset}" rpy="0.0 0.0 0.0" />             -->
+                        xyz="0.0 0.0 ${base_link_inertia_z_offset}" rpy="0.0 0.0 0.0" />             -->
     </link>
     <!-- footprint_body_joint -->
     <joint name="footprint_body_joint" type="fixed">
-        <parent link="footprint_link"/>
-        <child link="body_link"/>
+        <parent link="base_footprint"/>
+        <child link="base_link"/>
         <origin xyz="0 0 ${caster_wheel_radius - body_caster_wheel_Achse_distance}" rpy= "0 0 0"/>
     </joint>
@@ -78,5 +78,5 @@
     <!-- body_left_wheel_joint -->
     <joint name="body_left_wheel_joint" type="continuous">
-        <parent link="body_link"/>
+        <parent link="base_link"/>
         <child link="left_wheel_link"/>
         <origin xyz="0.0 ${(wheel_x_offset + (wheel_length/2))} ${wheel_z_offset}" rpy= "${pi/2} 0.0 0.0"/>
@@ -85,5 +85,5 @@
     <!-- body_right_wheel_joint -->
     <joint name="body_right_wheel_joint" type="continuous">
-        <parent link="body_link"/>
+        <parent link="base_link"/>
         <child link="right_wheel_link"/>
         <origin xyz="0.0 ${-(wheel_x_offset + (wheel_length/2))} ${wheel_z_offset}" rpy= "${pi/2} 0.0 0.0"/>
@@ -138,5 +138,5 @@
     <!--body_front_caster_wheel_joint-->
     <joint name="body_front_caster_wheel_joint" type="fixed">
-        <parent link="body_link"/>
+        <parent link="base_link"/>
         <child link="front_caster_wheel_link"/>
         <origin xyz="${-body_caster_wheel_link_distance} 0.0 ${-(body_caster_wheel_Achse_distance + 0.001)}" rpy="0.0 ${pi/2} 0.0"/>
@@ -144,5 +144,5 @@
     <!--body_rear_caster_wheel_joint-->
     <joint name="body_rear_caster_wheel_joint" type="fixed">
-        <parent link="body_link"/>
+        <parent link="base_link"/>
         <child link="rear_caster_wheel_link"/>
         <origin xyz="${body_caster_wheel_link_distance} 0.0 ${-(body_caster_wheel_Achse_distance + 0.001)}" rpy="0.0 ${pi/2} 0.0"/>

File: src/my_robot_description/urdf/my_robot_base_mesh.xacro (robot description, xacro)
@@ -1,16 +1,16 @@
 <?xml version="1.0"?>
 <robot xmlns:xacro="http://www.ros.org/wiki/xacro">
-    <xacro:property name="wheel_y_offset" value="0.075"/>
+    <xacro:property name="wheel_y_offset" value="0.0775"/>
     <xacro:property name="wheel_z_offset" value="0.02"/>
     <xacro:property name="wheel_radius" value="0.0325"/>
     <xacro:property name="wheel_length" value="0.025"/>
-    <xacro:property name="robot_center_to_body_link_x_distance" value="0.054"/>
-    <xacro:property name="robot_center_to_body_link_z_distance" value="0.1375"/>
+    <xacro:property name="robot_center_to_base_link_x_distance" value="0.054"/>
+    <xacro:property name="robot_center_to_base_link_z_distance" value="0.1375"/>
     <xacro:property name="body_length" value="0.1855"/>
     <xacro:property name="body_radius" value="0.07"/>
     <xacro:property name="caster_wheel_radius" value="0.0125"/>
     <xacro:property name="caster_wheel_length" value="0.013"/>
-    <xacro:property name="body_caster_wheel_link_distance" value="0.0485"/>
-    <xacro:property name="body_link_inertia_z_offset" value="0.0925"/>
+    <xacro:property name="base_caster_wheel_link_distance" value="0.0485"/>
+    <xacro:property name="base_link_inertia_z_offset" value="0.0925"/>
     <xacro:property name="lidar_radius" value="0.0278"/>
     <xacro:property name="lidar_length" value="0.0413"/>
@@ -18,15 +18,15 @@
     <xacro:property name="imu_width" value="0.02"/>
     <xacro:property name="imu_height" value="0.002"/>
-    <xacro:property name="body_imu_z_distance" value="${body_length - 0.046}"/>
-    <!-- footprint_link -->
-    <link name="footprint_link" />
-    <!-- body_link -->
-    <link name="body_link">
+    <xacro:property name="base_imu_z_distance" value="${body_length - 0.046}"/>
+    <!-- base_footprint -->
+    <link name="base_footprint" />
+    <!-- base_link -->
+    <link name="base_link">
         <visual>
             <geometry>
-                <mesh filename="package://my_robot_description/meshes_description/my_robot.stl" scale="0.001 0.001 0.001"/>
+                <mesh filename="package://my_robot_description/meshes_description/my_robot_1.stl" scale="0.001 0.001 0.001"/>
             </geometry>
             <material name="grey"/>
-            <origin xyz="0.0 0.0 ${robot_center_to_body_link_z_distance}" rpy="${pi/2} 0.0 ${pi/2}"/>
+            <origin xyz="0.0 0.0 ${robot_center_to_base_link_z_distance}" rpy="${pi/2} 0.0 ${pi/2}"/>
         </visual>
         <collision>
@@ -39,8 +39,8 @@
                                 xyz="0.0 0.0 ${wheel_z_offset + (body_length / 2) - 0.02}" rpy="0.0 0.0 0.0" />
     </link>
-    <!-- footprint_body_joint -->
-    <joint name="footprint_body_joint" type="fixed">
-        <parent link="footprint_link"/>
-        <child link="body_link"/>
+    <!-- footprint_base_joint -->
+    <joint name="footprint_base_joint" type="fixed">
+        <parent link="base_footprint"/>
+        <child link="base_link"/>
         <origin xyz="0 0 ${caster_wheel_radius}" rpy= "0 0 0"/>
     </joint>
@@ -67,14 +67,14 @@
     <xacro:wheel_link prefix="right"/>
     <xacro:wheel_link prefix="left"/>
-    <!-- body_left_wheel_joint -->
-    <joint name="body_left_wheel_joint" type="continuous">
-        <parent link="body_link"/>
+    <!-- base_left_wheel_joint -->
+    <joint name="base_left_wheel_joint" type="continuous">
+        <parent link="base_link"/>
         <child link="left_wheel_link"/>
         <origin xyz="0.0 ${wheel_y_offset} ${wheel_z_offset}" rpy= "0.0 ${pi/2} ${pi/2}"/>
         <axis xyz="0 0 1"/>
     </joint>
-    <!-- body_right_wheel_joint -->
-    <joint name="body_right_wheel_joint" type="continuous">
-        <parent link="body_link"/>
+    <!-- base_right_wheel_joint -->
+    <joint name="base_right_wheel_joint" type="continuous">
+        <parent link="base_link"/>
         <child link="right_wheel_link"/>
         <origin xyz="0.0 ${-wheel_y_offset} ${wheel_z_offset}" rpy= "0.0 ${pi/2} ${pi/2}"/>
@@ -104,27 +104,27 @@
     <xacro:caster_wheel_link prefix="front"/>
     <xacro:caster_wheel_link prefix="rear"/>
-    <!--body_front_caster_wheel_joint-->
-    <joint name="body_front_caster_wheel_joint" type="fixed">
-        <parent link="body_link"/>
+    <!--base_front_caster_wheel_joint-->
+    <joint name="base_front_caster_wheel_joint" type="fixed">
+        <parent link="base_link"/>
         <child link="front_caster_wheel_link"/>
-        <origin xyz="${body_caster_wheel_link_distance} 0.0 0.00017" rpy= "0.0 ${pi/2} ${pi/2}"/>
+        <origin xyz="${base_caster_wheel_link_distance} 0.0 0.00017" rpy= "0.0 ${pi/2} ${pi/2}"/>
     </joint>
-    <!--body_rear_caster_wheel_joint-->
-    <joint name="body_rear_caster_wheel_joint" type="fixed">
-        <parent link="body_link"/>
+    <!--base_rear_caster_wheel_joint-->
+    <joint name="base_rear_caster_wheel_joint" type="fixed">
+        <parent link="base_link"/>
         <child link="rear_caster_wheel_link"/>
-        <origin xyz="${-body_caster_wheel_link_distance} 0.0 0.00017" rpy="0.0 ${pi/2} ${pi/2}"/>
+        <origin xyz="${-base_caster_wheel_link_distance} 0.0 0.00017" rpy="0.0 ${pi/2} ${pi/2}"/>
     </joint>
     <!-- odom_link -->
     <!-- <link name="odom" /> -->
-    <!-- body_link_odom_joint -->
+    <!-- base_link_odom_joint -->
     <!-- <joint name="odom_joint" type="fixed">
         <parent link="odom"/>
-        <child link="body_link"/>
+        <child link="base_link"/>
         <origin xyz="0 0 0" rpy="0 0 0"/>
     </joint> -->
-    <!-- body_link_Joint
-    <joint name="laser_joint" type="fixed">
-        <parent link="body_link"/>
+    <!-- base_link_Joint -->
+    <!-- <joint name="laser_joint" type="fixed">
+        <parent link="base_link"/>
         <child link="laser"/>
         <origin xyz="0 0 0.1" rpy="0 0 0"/>

File: src/my_robot_description/urdf/my_robot_gazebo_control.xacro (robot description, xacro)
@@ -11,5 +11,5 @@
             <right_joint>body_right_wheel_joint</right_joint>
             <!-- kinematics -->
-            <wheel_separation>0.127</wheel_separation>
+            <wheel_separation>0.155</wheel_separation>
             <wheel_diameter>0.065</wheel_diameter>
             <!-- limits -->
@@ -26,5 +26,5 @@
             <!-- <odometry_source>world</odometry_source> -->
             <publish_tf>true</publish_tf>
-            <robot_base_frame>footprint_link</robot_base_frame>
+            <robot_base_frame>base_footprint</robot_base_frame>
         </plugin>
     </gazebo>

File: src/my_robot_description/urdf/my_robot_ros2_control.xacro (robot description, xacro)
@@ -4,6 +4,10 @@
         <hardware>
             <plugin>gazebo_ros2_control/GazeboSystem</plugin>
+            <!-- ros2-control Real Robot -->
+            <!-- <plugin>my_robot_control/MyRobotInterface</plugin>
+            <param name="port">/dev/esp32</param> -->
         </hardware>
-        <joint name="body_left_wheel_joint">
+        <!-- ros2_control Interfaces -->
+        <joint name="base_left_wheel_joint">
             <command_interface name="velocity">
                 <param name="min">-10</param>
@@ -13,5 +17,5 @@
             <state_interface name="position"/>
         </joint>
-        <joint name="body_right_wheel_joint">
+        <joint name="base_right_wheel_joint">
             <command_interface name="velocity">
                 <param name="min">-10</param>
@@ -22,7 +26,14 @@
         </joint>
     </ros2_control>
-    <!-- <ros2_control name="GazeboSystem" type="system">
+    <!-- <ros2_control name="DiffDriveSystem" type="system">
         <hardware>
-            <plugin>gazebo_ros2_control/GazeboSystem</plugin>
+            <plugin>diffbot_hardware_interface/DiffDriveHardwareInterface</plugin>
+            <param name="left_wheel_name">left_wheel_joint</param>
+            <param name="right_wheel_name">right_wheel_joint</param>
+            <param name="loop_rate">30</param>
+            <param name="device">/dev/esp</param>
+            <param name="baud_rate">57600</param>
+            <param name="timeout">1000</param>
+            <param name="enc_counts_per_rev">960</param>
         </hardware>
         <joint name="body_left_wheel_joint">
@@ -62,6 +73,6 @@
             <robot_param_node>robot_state_publisher</robot_param_node>
             <parameters>$(find my_robot_description)/config/my_controllers.yaml</parameters>
-            <publish_tf>true</publish_tf>
-            <robot_base_frame>footprint_link</robot_base_frame>
+            <publish_tf>flase</publish_tf>
+            <robot_base_frame>base_footprint</robot_base_frame>
         </plugin>
     </gazebo>
