Commit message: added stl-Files and modifed urdf-datei

File: src/my_robot_description/urdf/common_properties.xacro (robot description, xacro)
@@ -19,4 +19,16 @@
         <color rgba="0.0 0.1 0.0 1"/>
     </material>
+    <material name="grünlichesGrau">
+        <color rgba="0.6 0.7 0.6 1"/>
+    </material>
+<material name="warmesRot">
+    <color rgba="0.8 0.1 0.1 1"/>
+</material>
+<material name="grauBlau">
+    <color rgba="0.4 0.5 0.6 1"/>
+</material>
+<material name="pastelligesZitronengelb">
+    <color rgba="1.0 1.0 0.6 1"/>
+</material>
     <gazebo reference="base_link">
         <material>Gazebo/DarkGrey</material>

File: src/my_robot_description/urdf/imu.xacro (robot description, xacro)
@@ -5,14 +5,15 @@
         <visual>
             <geometry>
-                <box size="${imu_length} ${imu_width} ${imu_height}"/>
+                <mesh filename="package://my_robot_description/models/meshes/adafruit_bno055_stemma_qt_1.stl" scale="0.001 0.001 0.001"/>
+                <!-- <box size="${imu_length} ${imu_width} ${imu_height}"/> -->
             </geometry>
-            <material name="green"/>
-            <origin xyz="0.0 0.0 ${imu_height/2}" rpy="0.0 0.0 ${pi/2}"/>
+            <material name="warmesRot"/>
+            <origin xyz="0.0 0.0 ${imu_height/2}" rpy="0.0 0.0 0.0"/>
         </visual>
         <collision>
             <geometry>
-                <box size="${imu_length} ${imu_width} ${imu_height}"/>
+                <box size="${imu_width} ${imu_length} ${imu_height * 3}"/>
             </geometry>
-            <origin xyz="0.0 0.0 ${imu_height/2}" rpy="0.0 0.0 ${pi/2}"/>
+            <origin xyz="0.0 0.0 ${imu_height * 2}" rpy="0.0 0.0 ${pi/2}"/>
         </collision>
         <xacro:box_inertia m="0.05" l="${imu_length}" w="${imu_width}" h="${imu_height}"
@@ -23,10 +24,9 @@
         <parent link="base_link"/>
         <child link="bno055"/>
-        <origin xyz="0 0 ${base_imu_z_distance + 0.0345}" rpy= "0 0 0"/>
+        <origin xyz="0 0 ${base_imu_z_distance + 0.0335}" rpy= "0 0 0.0"/>
     </joint>
-    <gazebo reference="bno055">
+    <!-- <gazebo reference="bno055">
         <material>Gazebo/Red</material>
         <sensor name="bno055" type="imu">
-            <!-- ensure the sensor is active (required) -->
             <always_on>true</always_on>
             <update_rate>100</update_rate>
@@ -35,5 +35,4 @@
             <plugin name="bno055_plugin" filename="libgazebo_ros_imu_sensor.so">
                 <ros>
-                    <!-- publish to /imu/data -->
                     <namespace>/imu</namespace>
                     <remapping>~/out:=/imu/data</remapping>
@@ -84,4 +83,4 @@
             </imu>
         </sensor>
-    </gazebo>
+    </gazebo> -->
 </robot>

File: src/my_robot_description/urdf/lidar.xacro (robot description, xacro)
@@ -5,14 +5,17 @@
         <visual>
             <geometry>
-                <cylinder radius="${lidar_radius}" length="${lidar_length}"/>
+                <mesh filename="package://my_robot_description/models/meshes/c1m1_appearance_v2_20230926_3d_.stl" scale="0.001 0.001 0.001"/>
+                <!-- <cylinder radius="${lidar_radius}" length="${lidar_length}"/> -->
             </geometry>
-            <material name="red"/>
-            <origin xyz="0.0 0.0 ${lidar_length/2}" rpy="0.0 0.0 0.0"/>
+            <material name="pastelligesZitronengelb"/>
+            <origin xyz="0.0 0.0 0.0" rpy="0.0 0.0 0.0"/>
+            <!-- <origin xyz="0.0 0.0 ${lidar_length/2}" rpy="0.0 0.0 0.0"/>           -->
         </visual>
         <collision>
             <geometry>
-                <cylinder radius="${lidar_radius}" length="${lidar_length}"/>
+                <cylinder radius="${lidar_radius + 0.007}" length="${lidar_length}"/>
             </geometry>
             <origin xyz="0.0 0.0 ${lidar_length/2}" rpy="0.0 0.0 0.0"/>
+            <!-- <origin xyz="0.0 0.0 ${lidar_length/2}" rpy="0.0 0.0 0.0"/>                    -->
         </collision>
         <xacro:cylinder_inertia m="0.1" r="${lidar_radius}" h="${lidar_length - 0.002}"

File: src/my_robot_description/urdf/my_robot.urdf.xacro (robot description, xacro)
@@ -6,8 +6,9 @@
     <!-- <xacro:include filename="my_robot_base.xacro" /> -->
     <xacro:include filename="my_robot_base_mesh.xacro" />
+    <!-- <xacro:include filename="my_robot_base_mesh.urdf" /> -->
     <xacro:include filename="lidar.xacro" />
     <xacro:include filename="imu.xacro" />
+    <!-- <xacro:include filename="my_robot_ros2_control.xacro" />   -->
     <!-- <xacro:include filename="my_robot_gazebo_control.xacro" /> -->
-    <!-- <xacro:include filename="my_robot_ros2_control.xacro" />   -->
     <!-- <xacro:if value="$(arg use_ros2_control)">
         <xacro:include filename="my_robot_ros2_control.xacro" />

File: src/my_robot_description/urdf/my_robot_base.xacro (robot description, xacro)
@@ -1,19 +1,22 @@
 <?xml version="1.0"?>
 <robot xmlns:xacro="http://www.ros.org/wiki/xacro">
-    <xacro:property name="wheel_x_offset" value="0.045"/>
-    <xacro:property name="wheel_z_offset" value="0.0225"/>
+    <xacro:property name="wheel_y_offset" value="0.0775"/>
+    <xacro:property name="wheel_z_offset" value="0.02"/>
     <xacro:property name="wheel_radius" value="0.0325"/>
     <xacro:property name="wheel_length" value="0.025"/>
+    <xacro:property name="robot_center_to_base_link_x_distance" value="0.054"/>
     <xacro:property name="robot_center_to_base_link_z_distance" value="0.1375"/>
     <xacro:property name="body_length" value="0.1855"/>
     <xacro:property name="body_radius" value="0.07"/>
-    <xacro:property name="body_width" value="0.1"/>
     <xacro:property name="caster_wheel_radius" value="0.0125"/>
     <xacro:property name="caster_wheel_length" value="0.013"/>
-    <xacro:property name="body_caster_wheel_link_distance" value="0.06"/>
-    <xacro:property name="body_caster_wheel_Achse_distance" value="0.0025"/>
+    <xacro:property name="base_caster_wheel_link_distance" value="0.0485"/>
     <xacro:property name="base_link_inertia_z_offset" value="0.0925"/>
     <xacro:property name="lidar_radius" value="0.0278"/>
     <xacro:property name="lidar_length" value="0.0413"/>
+    <xacro:property name="imu_length" value="0.015"/>
+    <xacro:property name="imu_width" value="0.02"/>
+    <xacro:property name="imu_height" value="0.0015"/>
+    <xacro:property name="base_imu_z_distance" value="${body_length - 0.046}"/>
     <!-- base_footprint -->
     <link name="base_footprint" />
@@ -22,35 +25,23 @@
         <visual>
             <geometry>
-                <box size="${body_radius * 2} ${body_radius * 2} ${body_length}"/>
-                <!-- <mesh filename="package://my_robot/meshes_description/my_robot.stl" scale="0.001 0.001 0.001"/> -->
+                <mesh filename="package://my_robot_description/models/meshes/my_robot_base.stl" scale="0.001 0.001 0.001"/>
             </geometry>
             <material name="grey"/>
-            <origin xyz="0.0 0.0 ${wheel_z_offset + (body_length / 2) - 0.02}" rpy="0.0 0.0 0.0"/>
-            <!-- <origin xyz="0.0 0.0 ${robot_center_to_base_link_z_distance}" rpy="${pi/2} 0.0 0.0"/>           -->
+            <origin xyz="0.0 0.0 ${robot_center_to_base_link_z_distance}" rpy="${pi/2} 0.0 ${pi/2}"/>
         </visual>
         <collision>
             <geometry>
-                <box size="${body_radius * 2} ${body_radius * 2} ${body_length}"/>
-                <!-- <box size="${body_radius * 2} ${(body_radius * 2) - wheel_length} ${body_length}"/> -->
+                <cylinder radius="${body_radius}" length="${body_length}"/>
             </geometry>
-            <origin xyz="0.0 0.0 ${wheel_z_offset + (body_length / 2) - 0.02}" rpy="0.0 0.0 0.0"/>
-            <!-- <origin xyz="0.0 0.0 ${robot_center_to_base_link_z_distance}" rpy="${pi/2} 0.0 0.0"/>                    -->
+            <origin xyz="0.0 0.0 ${body_length / 2}" rpy="0.0 0.0 0.0"/>
         </collision>
-        <!-- <collision>
-            <geometry>
-                <mesh filename="package://my_robot/meshes_description/my_robot.stl" scale="0.001 0.001 0.001"/>
-            </geometry>
-            <origin xyz="0.0 0.0 ${robot_center_to_base_link_z_distance}" rpy="${pi/2} 0.0 0.0"/>
-        </collision> -->
-        <xacro:box_inertia m="10.0" l="${body_length}" w="${body_radius * 2}" h="${wheel_x_offset * 2}"
+        <xacro:box_inertia m="1000.0" l="${body_length}" w="${body_radius * 2}" h="${body_radius * 2}"
                                 xyz="0.0 0.0 ${wheel_z_offset + (body_length / 2) - 0.02}" rpy="0.0 0.0 0.0" />
-        <!-- <xacro:cylinder_inertia m="1.5" r="${body_radius}" h="${body_length}"
-                        xyz="0.0 0.0 ${base_link_inertia_z_offset}" rpy="0.0 0.0 0.0" />             -->
     </link>
-    <!-- footprint_body_joint -->
-    <joint name="footprint_body_joint" type="fixed">
+    <!-- footprint_base_joint -->
+    <joint name="footprint_base_joint" type="fixed">
         <parent link="base_footprint"/>
         <child link="base_link"/>
-        <origin xyz="0 0 ${caster_wheel_radius - body_caster_wheel_Achse_distance}" rpy= "0 0 0"/>
+        <origin xyz="0 0 ${caster_wheel_radius}" rpy= "0 0 0"/>
     </joint>
     <!-- wheel_link -->
@@ -66,9 +57,9 @@
             <collision>
                 <geometry>
-                    <cylinder radius="${wheel_radius}" length="${wheel_length}"/>
+                    <sphere radius="${wheel_radius}"/>
                 </geometry>
                 <origin xyz="0.0 0.0 0.0" rpy="0.0 0.0 0.0"/>
             </collision>
-            <xacro:cylinder_inertia m="2.0" r="${wheel_radius}" h="${wheel_length}"
+            <xacro:cylinder_inertia m="500.0" r="${wheel_radius}" h="${wheel_length}"
                                     xyz="0.0 0.0 0.0" rpy="0.0 0.0 0.0" />
         </link>
@@ -76,43 +67,20 @@
     <xacro:wheel_link prefix="right"/>
     <xacro:wheel_link prefix="left"/>
-    <!-- body_left_wheel_joint -->
-    <joint name="body_left_wheel_joint" type="continuous">
+    <!-- base_left_wheel_joint -->
+    <joint name="base_left_wheel_joint" type="continuous">
         <parent link="base_link"/>
         <child link="left_wheel_link"/>
-        <origin xyz="0.0 ${(wheel_x_offset + (wheel_length/2))} ${wheel_z_offset}" rpy= "${pi/2} 0.0 0.0"/>
-        <axis xyz="0 0 -1"/>
+        <origin xyz="0.0 ${wheel_y_offset} ${wheel_z_offset}" rpy= "0.0 ${pi/2} ${pi/2}"/>
+        <axis xyz="0 0 1"/>
     </joint>
-    <!-- body_right_wheel_joint -->
-    <joint name="body_right_wheel_joint" type="continuous">
+    <!-- base_right_wheel_joint -->
+    <joint name="base_right_wheel_joint" type="continuous">
         <parent link="base_link"/>
         <child link="right_wheel_link"/>
-        <origin xyz="0.0 ${-(wheel_x_offset + (wheel_length/2))} ${wheel_z_offset}" rpy= "${pi/2} 0.0 0.0"/>
-        <axis xyz="0 0 -1"/>
+        <origin xyz="0.0 ${-wheel_y_offset} ${wheel_z_offset}" rpy= "0.0 ${pi/2} ${pi/2}"/>
+        <axis xyz="0 0 1"/>
     </joint>
-    <!-- caster-Wheel-link-sphere-->
+    <!-- caster-Wheel-link -->
     <xacro:macro name="caster_wheel_link" params="prefix">
-        <link name="${prefix}_caster_wheel_link">
-            <visual>
-                <geometry>
-                    <sphere radius="${caster_wheel_radius / 2}"/>
-                </geometry>
-                <material name="red"/>
-                <origin xyz="0.0 0.0 0.0" rpy="0.0 0.0 0.0"/>
-            </visual>
-            <collision>
-                <geometry>
-                    <sphere radius="${caster_wheel_radius / 2}"/>
-                </geometry>
-                <material name="black"/>
-                <origin xyz="0.0 0.0 0.0" rpy="0.0 0.0 0.0"/>
-            </collision>
-            <xacro:sphere_inertia m="0.1" r="${caster_wheel_radius / 2}"
-                                    xyz="0.0 0.0 0.0" rpy="0.0 0.0 0.0" />
-        </link>
-    </xacro:macro>
-    <xacro:caster_wheel_link prefix="front"/>
-    <xacro:caster_wheel_link prefix="rear"/>
-    <!-- caster-Wheel-link-cylinder-->
-    <!-- <xacro:macro name="caster_wheel_link" params="prefix">
         <link name="${prefix}_caster_wheel_link">
             <visual>
@@ -121,30 +89,44 @@
                 </geometry>
                 <material name="black"/>
-                <origin xyz="0.0 0.0 0.0" rpy="0.0 0.0 0.0"/>
+                <origin xyz="0.0 0.0 0.0" rpy="0.0 0.0  0.0"/>
             </visual>
             <collision>
                 <geometry>
-                    <cylinder radius="${caster_wheel_radius}" length="${caster_wheel_length}"/>
+                    <sphere radius="${caster_wheel_radius}"/>
                 </geometry>
                 <material name="black"/>
                 <origin xyz="0.0 0.0 0.0" rpy="0.0 0.0 0.0"/>
             </collision>
-            <xacro:cylinder_inertia m="0.05" r="${caster_wheel_radius + 0.0019}" h="${caster_wheel_length}"
+            <xacro:cylinder_inertia m="250.0" r="${caster_wheel_radius}" h="${caster_wheel_length}"
                                     xyz="0.0 0.0 0.0" rpy="0.0 0.0 0.0" />
         </link>
     </xacro:macro>
     <xacro:caster_wheel_link prefix="front"/>
-    <xacro:caster_wheel_link prefix="rear"/> -->
-    <!--body_front_caster_wheel_joint-->
-    <joint name="body_front_caster_wheel_joint" type="fixed">
+    <xacro:caster_wheel_link prefix="rear"/>
+    <!--base_front_caster_wheel_joint-->
+    <joint name="base_front_caster_wheel_joint" type="fixed">
         <parent link="base_link"/>
         <child link="front_caster_wheel_link"/>
-        <origin xyz="${-body_caster_wheel_link_distance} 0.0 ${-(body_caster_wheel_Achse_distance + 0.001)}" rpy="0.0 ${pi/2} 0.0"/>
+        <origin xyz="${base_caster_wheel_link_distance} 0.0 0.00017" rpy="0.0 ${pi/2} ${pi/2}"/>
     </joint>
-    <!--body_rear_caster_wheel_joint-->
-    <joint name="body_rear_caster_wheel_joint" type="fixed">
+    <!--base_rear_caster_wheel_joint-->
+    <joint name="base_rear_caster_wheel_joint" type="fixed">
         <parent link="base_link"/>
         <child link="rear_caster_wheel_link"/>
-        <origin xyz="${body_caster_wheel_link_distance} 0.0 ${-(body_caster_wheel_Achse_distance + 0.001)}" rpy="0.0 ${pi/2} 0.0"/>
+        <origin xyz="${-base_caster_wheel_link_distance} 0.0 0.00017" rpy="0.0 ${pi/2} ${pi/2}"/>
     </joint>
+    <!-- odom_link -->
+    <!-- <link name="odom" /> -->
+    <!-- base_link_odom_joint -->
+    <!-- <joint name="odom_joint" type="fixed">
+        <parent link="odom"/>
+        <child link="base_link"/>
+        <origin xyz="0 0 0" rpy="0 0 0"/>
+    </joint> -->
+    <!-- base_link_Joint -->
+    <!-- <joint name="laser_joint" type="fixed">
+        <parent link="base_link"/>
+        <child link="laser"/>
+        <origin xyz="0 0 0.1" rpy="0 0 0"/>
+    </joint> -->
 </robot>

File: src/my_robot_description/urdf/my_robot_base_mesh.xacro (robot description, xacro)
@@ -2,6 +2,6 @@
 <robot xmlns:xacro="http://www.ros.org/wiki/xacro">
     <xacro:property name="wheel_y_offset" value="0.0775"/>
-    <xacro:property name="wheel_z_offset" value="0.02"/>
-    <xacro:property name="wheel_radius" value="0.0325"/>
+    <xacro:property name="wheel_z_offset" value="0.0205"/>
+    <xacro:property name="wheel_radius" value="0.033"/>
     <xacro:property name="wheel_length" value="0.025"/>
     <xacro:property name="robot_center_to_base_link_x_distance" value="0.054"/>
@@ -15,7 +15,7 @@
     <xacro:property name="lidar_radius" value="0.0278"/>
     <xacro:property name="lidar_length" value="0.0413"/>
-    <xacro:property name="imu_length" value="0.015"/>
+    <xacro:property name="imu_length" value="0.025"/>
     <xacro:property name="imu_width" value="0.02"/>
-    <xacro:property name="imu_height" value="0.002"/>
+    <xacro:property name="imu_height" value="0.0015"/>
     <xacro:property name="base_imu_z_distance" value="${body_length - 0.046}"/>
     <!-- base_footprint -->
@@ -25,7 +25,7 @@
         <visual>
             <geometry>
-                <mesh filename="package://my_robot_description/meshes_description/my_robot_1.stl" scale="0.001 0.001 0.001"/>
+                <mesh filename="package://my_robot_description/models/meshes/my_robot_base.stl" scale="0.001 0.001 0.001"/>
             </geometry>
-            <material name="grey"/>
+            <material name="grünlichesGrau"/>
             <origin xyz="0.0 0.0 ${robot_center_to_base_link_z_distance}" rpy="${pi/2} 0.0 ${pi/2}"/>
         </visual>
@@ -50,8 +50,8 @@
             <visual>
                 <geometry>
-                    <cylinder radius="${wheel_radius}" length="${wheel_length}"/>
+                <mesh filename="package://my_robot_description/models/meshes/wheel.stl" scale="0.001 0.001 0.001"/>
                 </geometry>
-                <material name="orange"/>
-                <origin xyz="0.0 0.0 0.0" rpy="0.0 0.0 0.0"/>
+                <material name="grauBlau"/>
+                <origin xyz="0.0 0.0 ${-wheel_length/2}" rpy="${pi/2}  0.0 0.0"/>
             </visual>
             <collision>
@@ -71,6 +71,6 @@
         <parent link="base_link"/>
         <child link="left_wheel_link"/>
-        <origin xyz="0.0 ${wheel_y_offset} ${wheel_z_offset}" rpy= "0.0 ${pi/2} ${pi/2}"/>
-        <axis xyz="0 0 1"/>
+        <origin xyz="0.0 ${wheel_y_offset} ${wheel_z_offset}" rpy= "${-pi/2} ${pi} ${pi}"/>
+        <axis xyz="0 0 -1"/>
     </joint>
     <!-- base_right_wheel_joint -->
@@ -78,5 +78,5 @@
         <parent link="base_link"/>
         <child link="right_wheel_link"/>
-        <origin xyz="0.0 ${-wheel_y_offset} ${wheel_z_offset}" rpy= "0.0 ${pi/2} ${pi/2}"/>
+        <origin xyz="0.0 ${-wheel_y_offset} ${wheel_z_offset}" rpy= "${-pi/2} 0.0 0.0"/>
         <axis xyz="0 0 1"/>
     </joint>
@@ -86,8 +86,8 @@
             <visual>
                 <geometry>
-                    <cylinder radius="${caster_wheel_radius}" length="${caster_wheel_length}"/>
+                    <mesh filename="package://my_robot_description/models/meshes/caster_wheel.stl" scale="0.001 0.001 0.001"/>
                 </geometry>
                 <material name="black"/>
-                <origin xyz="0.0 0.0 0.0" rpy="0.0 0.0  0.0"/>
+                <origin xyz="0.0 ${caster_wheel_length/2} 0.0" rpy="0.0 0.0 ${-pi/2}"/>
             </visual>
             <collision>
@@ -108,5 +108,5 @@
         <parent link="base_link"/>
         <child link="front_caster_wheel_link"/>
-        <origin xyz="${base_caster_wheel_link_distance} 0.0 0.00017" rpy= "0.0 ${pi/2} ${pi/2}"/>
+        <origin xyz="${base_caster_wheel_link_distance} 0.0 0.00017" rpy= "0.0 0.0 0.0"/>
     </joint>
     <!--base_rear_caster_wheel_joint-->
@@ -114,5 +114,5 @@
         <parent link="base_link"/>
         <child link="rear_caster_wheel_link"/>
-        <origin xyz="${-base_caster_wheel_link_distance} 0.0 0.00017" rpy="0.0 ${pi/2} ${pi/2}"/>
+        <origin xyz="${-base_caster_wheel_link_distance} 0.0 0.00017" rpy= "0.0 0.0 0.0"/>
     </joint>
     <!-- odom_link -->
@@ -121,5 +121,5 @@
     <!-- <joint name="odom_joint" type="fixed">
         <parent link="odom"/>
-        <child link="base_link"/>
+        <child link="base_footprint"/>
         <origin xyz="0 0 0" rpy="0 0 0"/>
     </joint> -->

File: src/my_robot_description/urdf/my_robot_gazebo_control.xacro (robot description, xacro)
@@ -8,6 +8,6 @@
             <num_wheel_pairs>1</num_wheel_pairs>
             <!-- whell Information -->
-            <left_joint>body_left_wheel_joint</left_joint>
-            <right_joint>body_right_wheel_joint</right_joint>
+            <left_joint>base_left_wheel_joint</left_joint>
+            <right_joint>base_right_wheel_joint</right_joint>
             <!-- kinematics -->
             <wheel_separation>0.155</wheel_separation>

File: src/my_robot_description/urdf/my_robot_ros2_control.xacro (robot description, xacro)
@@ -37,5 +37,5 @@
             <param name="enc_counts_per_rev">960</param>
         </hardware>
-        <joint name="body_left_wheel_joint">
+        <joint name="base_left_wheel_joint">
             <command_interface name="velocity">
                 <param name="min">-10</param>
@@ -45,5 +45,5 @@
             <state_interface name="position"/>
         </joint>
-        <joint name="body_right_wheel_joint">
+        <joint name="base_right_wheel_joint">
             <command_interface name="velocity">
                 <param name="min">-10</param>
@@ -64,5 +64,5 @@
         <plugin>transmission_interface/SimpleTransmission</plugin>
         <actuator name="left_wheel_motor" role="actuator_left"/>
-        <joint name="body_left_wheel_joint" role="joint_left">
+        <joint name="base_left_wheel_joint" role="joint_left">
             <mechanical_reduction>2.0</mechanical_reduction>
         </joint>
@@ -73,5 +73,5 @@
             <robot_param_node>robot_state_publisher</robot_param_node>
             <parameters>$(find my_robot_description)/config/my_controllers.yaml</parameters>
-            <publish_tf>flase</publish_tf>
+            <publish_tf>false</publish_tf>
             <robot_base_frame>base_footprint</robot_base_frame>
         </plugin>
