Commit message: Add camera_link to my_robot_description pkg

File: src/my_robot_description/urdf/common_properties.xacro (robot description, xacro)
@@ -22,13 +22,13 @@
         <color rgba="0.6 0.7 0.6 1"/>
     </material>
-<material name="warmesRot">
-    <color rgba="0.8 0.1 0.1 1"/>
-</material>
-<material name="grauBlau">
-    <color rgba="0.4 0.5 0.6 1"/>
-</material>
-<material name="pastelligesZitronengelb">
-    <color rgba="1.0 1.0 0.6 1"/>
-</material>
+    <material name="warmesRot">
+        <color rgba="0.8 0.1 0.1 1"/>
+    </material>
+    <material name="grauBlau">
+        <color rgba="0.4 0.5 0.6 1"/>
+    </material>
+    <material name="pastelligesZitronengelb">
+        <color rgba="1.0 1.0 0.6 1"/>
+    </material>
     <gazebo reference="base_link">
         <material>Gazebo/DarkGrey</material>

File: src/my_robot_description/urdf/my_robot.urdf.xacro (robot description, xacro)
@@ -2,8 +2,7 @@
 <robot name="my_robot_description" xmlns:xacro="http://www.ros.org/wiki/xacro">
     <xacro:include filename="common_properties.xacro" />
-    <!-- <xacro:include filename="my_robot_base.xacro" /> -->
     <xacro:include filename="my_robot_base_mesh.xacro" />
-    <!-- <xacro:include filename="my_robot_base_mesh.urdf" /> -->
     <xacro:include filename="lidar.xacro" />
     <xacro:include filename="imu.xacro" />
+    <xacro:include filename="camera.xacro" />
 </robot>

File: src/my_robot_description/urdf/my_robot_base_mesh.urdf (robot description, URDF)
Before this commit: robot my_robot, 8 links, 7 joints
Links:
- added link camera, mass 0.05; collision box size=0.025 0.025 0.01; visual mesh filename=package://my_robot_description/models/meshes/cam_v2_1_v1.stl scale=0.001 0.001 0.001
- added link camera_optical
Joints:
- added joint base_camera_joint: type fixed, parent base_link, child camera, origin xyz=0.07 0 0.1465 rpy=0 0 0.0
- added joint camera_optical_joint: type fixed, parent camera, child camera_optical, origin xyz=0 0 0 rpy=-1.5707963267948966 0.0 -1.5707963267948966
